Commit message: Stand 20201203

File: innok_heros/innok_heros_description/urdf/innok_heros_4w.xacro (robot description, xacro)
@@ -15,20 +15,33 @@
   <xacro:property name="wheel_width"  value="0.160" />
   <xacro:property name="wheel_mass"   value="5.4" />
+  <!-- xacro:include filename="$(find innok_heros_description)/urdf/modules/heros_basefootprint.xacro" /-->
   <xacro:include filename="$(find innok_heros_description)/urdf/modules/heros_base_link.xacro"/>
-  <xacro:include filename="$(find innok_heros_description)/urdf/modules/heros_hokuyo.xacro"/>
+  <xacro:include filename="$(find innok_heros_description)/urdf/modules/sick_lms1xx.urdf.xacro"/>
   <xacro:include filename="$(find innok_heros_description)/urdf/modules/heros_wheel.xacro"/>
   <xacro:include filename="$(find innok_heros_description)/urdf/modules/heros_drive.xacro"/>
-  <xacro:include filename="$(find innok_heros_description)/urdf/modules/heros_caster.xacro"/>
   <xacro:include filename="$(find innok_heros_description)/urdf/modules/heros_battery.xacro"/>
-  <xacro:include filename="$(find innok_heros_description)/urdf/modules/heros_mounting_plate.xacro"/>
   <xacro:include filename="$(find innok_heros_description)/urdf/ROS/heros_joint_pub.xacro" />
   <xacro:include filename="$(find innok_heros_description)/urdf/ROS/heros_skid_drive.xacro" />
-  <heros_base_link   							/>
+  <!-- LiDar /-->
+  <xacro:sick_lms1xx
+	name="sick_lms1xx"
+	topic="scan"
+	joint="lms_joint"
+	frame="laser">
+  <origin xyz="5 0 -0.04" rpy="3.14 0 0"/>
+  </xacro:sick_lms1xx>
+  <xacro:sick_lms1xx
+	name="sick_lms1xx_back"
+	topic="scan_back"
+	joint="lms_joint_back"
+	frame="laser_back">
+  <origin xyz="-5.08 0 -0.04" rpy="3.14 0 3.14"/>
+  </xacro:sick_lms1xx>
+  <!--heros_basefootprint                                             /-->
+  <heros_base_link                                                />
   <heros_drive   	  front_rear='front'    dx='0.782' flip_z='-1'	/>
   <heros_drive   	  front_rear='rear'     dx='0.018' flip_z='1' 	/>
   <heros_battery 	  name='battery_box'    dx='0.336'		/>
-  <heros_mounting_plate   wheels='4'		dx='-0.02'		/>
   <heros_joint_pub joints='joint_base_wheel_rear_left, joint_base_wheel_rear_right, joint_base_wheel_front_left, joint_base_wheel_front_right'		/>
   <heros_skid_drive 							/>
-  <heros_hokuyo />
 </robot>

File: innok_heros/innok_heros_description/urdf/modules/heros_base_link.xacro (robot description, xacro)
@@ -20,6 +20,6 @@
     </inertial>
     <visual>
-      <origin xyz="0 0 0" rpy="0 0 0" />
-      <geometry> <mesh filename="package://innok_heros_description/meshes/beam.STL" /> </geometry>
+      <origin xyz="0.48 0 0" rpy="0 0 0" />
+      <geometry> <mesh filename="package://innok_heros_description/meshes/beam_02.STL" /> </geometry>
       <material name="white">
         <color rgba="1 1 1 1"/>
@@ -33,5 +33,5 @@
   <joint name="beam_joint" type="fixed">
     <origin
-      xyz="0 0 0" rpy="0 0 0" />
+      xyz="0 0 0.35" rpy="0 0 0" />
     <parent link="base_link" />
     <child link="beam_link" />

File: innok_heros/innok_heros_description/urdf/modules/heros_hokuyo.xacro (robot description, xacro)
@@ -40,5 +40,5 @@
     <sensor type="ray" name="sick_lms100_sensor">
       <pose>0 0 0 0 0 0</pose>
-      <visualize>true</visualize>
+      <visualize>false</visualize>
       <update_rate>25</update_rate>
       <ray>

Commit message: inn desc

File: innok_heros/innok_heros_description/urdf/innok_heros_4w.xacro (robot description, xacro)
@@ -18,4 +18,5 @@
   <xacro:include filename="$(find innok_heros_description)/urdf/modules/heros_base_link.xacro"/>
   <xacro:include filename="$(find innok_heros_description)/urdf/modules/sick_lms1xx.urdf.xacro"/>
+  <xacro:include filename="$(find innok_heros_description)/urdf/modules/imu.urdf.xacro"/>
   <xacro:include filename="$(find innok_heros_description)/urdf/modules/heros_wheel.xacro"/>
   <xacro:include filename="$(find innok_heros_description)/urdf/modules/heros_drive.xacro"/>
@@ -29,5 +30,5 @@
 	joint="lms_joint"
 	frame="laser">
-  <origin xyz="5 0 -0.04" rpy="3.14 0 0"/>
+  <origin xyz="1.02 0 -0.04" rpy="3.14 0 0"/>
   </xacro:sick_lms1xx>
   <xacro:sick_lms1xx
@@ -36,6 +37,11 @@
 	joint="lms_joint_back"
 	frame="laser_back">
-  <origin xyz="-5.08 0 -0.04" rpy="3.14 0 3.14"/>
+  <origin xyz="-0.06 0 -0.04" rpy="3.14 0 3.14"/>
   </xacro:sick_lms1xx>
+  <!-- imu /-->
+  <xacro:imu_sensor
+        parent="beam_link">
+  <origin xyz="0.08 0 0.041" rpy="0 0 0"/>
+  </xacro:imu_sensor>
   <!--heros_basefootprint                                             /-->
   <heros_base_link                                                />

Commit message: 20210304_01

File: innok_heros/innok_heros_description/urdf/innok_heros_4w.xacro (robot description, xacro)
@@ -19,4 +19,5 @@
   <xacro:include filename="$(find innok_heros_description)/urdf/modules/sick_lms1xx.urdf.xacro"/>
   <xacro:include filename="$(find innok_heros_description)/urdf/modules/imu.urdf.xacro"/>
+  <xacro:include filename="$(find innok_heros_description)/urdf/modules/_d435.urdf.xacro" />
   <xacro:include filename="$(find innok_heros_description)/urdf/modules/heros_wheel.xacro"/>
   <xacro:include filename="$(find innok_heros_description)/urdf/modules/heros_drive.xacro"/>
@@ -44,4 +45,12 @@
   <origin xyz="0.175 0 0.041" rpy="0 0 0"/>
   </xacro:imu_sensor>
+    <!-- Camera /-->
+  <xacro:sensor_d435
+	      name="camera"
+      	topics_ns="camera"
+      	parent="base_link"
+      	publish_pointcloud="true">
+  <origin xyz="1 0 0.08" rpy="0 0 0"/>
+  </xacro:sensor_d435>
   <!--heros_basefootprint                                             /-->
   <heros_base_link                                                />
